File: Microwave_clock_circuit/Microwave_clock.sch (KiCad schematic (older format))
At the start: 27 parts

Commit message: Maing schematic a bit less bad
Clean-up, better descriptions and removed all connection errors.
Parts:
- added J1: Conn_01x03_Male, symbol Connector:Conn_01x03_Male
- added J?: USB_B, symbol Connector:USB_B
- gave numbers to parts that had none: 27
Connections:
- net labels added: Dis_A, Dis_B, Dis_C, Dis_D, Dis_E, Dis_F, Dis_G
- net labels removed: 2022-01-14
- wire segments 68 -> 116
- no-connect marks 0 -> 28
Other:
- note added: "7 segment display \n& it's driver"
- note added: "I soldered wire (with male USB A plug on the other side of wire) directly to board. \nHere on shcematic i power input is represented by USB B conector but it can be any 5V power supply."
- note added: "So i used clock circuitry from broken analog battery powered clock (i will rever to this small circuit board as "clock module")and hacked \nit in with this circuit. It powers it with ~1.7 V and converts outputed by clock module 1.7 V\n pulses into 0 volt impulsed pulled up to VCC (5V)\nWARNNING ! :\nClock_VCC, Clock_GND and Clock_Output are connected to conector that is representing clock module,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"
- note added: "So, i don't have 7 segment display symbols so\n let's pretend those BAR's are 7 segments display \nand those 2 LEDs in middle are dots on display. \nPS. I'm not sure to what pins of 7 segment display dots \nare conected but if i remember corectly those were B and C.\n But that dosn't matter sicne it is probably be diferend \ndepending on display and i salvage mine from microwave oven board \nand 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"
- note removed: "7 segment display & it's driver"
- note removed: "So i used clock circuitry from broken analog battery powered clock (i will rever to this small circuit board as "clock module")and hacked \nit in with this circuit. It powers it with ~1.7 V and converts outputed by clock module 1.7 V\n pulses into 0 volt impulsed pulled up to VCC (5V)\nWARNNING ! :\nClock_VCC, Clock_GND and Clock_Output are used only here and are not used as Labels but used to sy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"
- note removed: "So, i don't have 7 segment display symbols and even with tutorial i'm not sure if i use buses corectly but i hope you get the idea.\nnumering starts with 3 and ends at 7, two dots in the middle of display are represented by 2 dieds and have "addres" 5 i.e. are like 5'th digit.\n"
- moved on the sheet: BAR1, BAR2, BAR3, BAR4, D2, D3, U2, U3
